File: CLOCK_IT/SD.kicad_sch (KiCad schematic)
At the start: 9 parts, among them U3 AW9523BTQR

Commit message: :fire: added camera pin an pinout naming
Parts:
- added C16, C17, C18: 4.7uF, symbol Device:C
- added R5: 10K, symbol Device:R
Connections:
- net AGND is gone; now on net GND: FPC1.2
- net Cam_D0 is gone; now on net GND: FPC1.24
- net DGND is gone; now on net GND: FPC1.15
- net DOVDD is gone; now on net Cam_3.3V: FPC1.11
- net AVDD: now also C17.1
- net GND: now also C16.2, C17.2, C18.2, R5.2
- net Cam_D1 renamed Cam_3.3V
- net Cam_3.3V: now also C16.1
- net FSIN renamed DVDD
- net DVDD: now also C18.1
- net HREF renamed Cam_HREF
- net PCLK renamed Cam_PCLK
- net PWDN renamed Cam_PWDN
- net Cam_PWDN: now also R5.1
- net RESETB renamed Cam_RESET
- net SIOC renamed SDA_I2C
- net SIOD renamed SDL_I2C
- net STROBE: no longer names the net of FPC1.1
- net VSYNC renamed Cam_VSYNC
- net XVCLK renamed Cam_XVCLK
- no-connect marks 5 -> 6
