File: CLOCK_IT/SD.kicad_sch (KiCad schematic)
At the start: 13 parts, among them U3 AW9523BTQR

Commit message: :white_check_mark: Connected i2c bus switch
Connections:
- net SDA_I2C renamed CAM_SDA
- net SDL_I2C renamed CAM_SCL
Changed lines of the file:
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@@
 		)
 	)
-	(global_label "SDA_I2C"
+	(hierarchical_label "CAM_SCL"
 		(shape input)
-		(at 256.54 31.75 180)
-		(fields_autoplaced yes)
+		(at 256.54 26.67 180)
 		(effects
 			(font
@@
 			(justify right)
 		)
-		(property "Intersheetrefs" "${INTERSHEET_REFS}"
-			(at 245.9348 31.75 0)
-			(effects
-				(font
-					(size 1.27 1.27)
-				)
-				(justify right)
-				(hide yes)
-			)
-		)
 	)
-	(global_label "SDL_I2C"
+	(hierarchical_label "CAM_SDA"
 		(shape input)
-		(at 256.54 26.67 180)
-		(fields_autoplaced yes)
+		(at 256.54 31.75 180)
 		(effects
 			(font
@@
 			(justify right)
 		)
-		(property "Intersheetrefs" "${INTERSHEET_REFS}"
-			(at 245.9953 26.67 0)
-			(effects
-				(font
-					(size 1.27 1.27)
-				)
-				(justify right)
-				(hide yes)
-			)
-		)
 	)

Commit message: :construction:added LCD connector,, completed connections
Changed lines of the file:
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@@
 	(paper "A4")
-	(junction
-		(at 21.59 74.93)
-		(diameter 0)
-		(color 0 0 0 0)
-	)
 	(junction
 		(at 240.03 57.15)
@@
 		(color 0 0 0 0)
 	)
+	(junction
+		(at 15.24 74.93)
+		(diameter 0)
+		(color 0 0 0 0)
+	)
 	(no_connect
 		(at 57.15 82.55)
@@
 	(wire
 		(pts
-			(xy 41.91 64.77) (xy 22.86 64.77)
-		)
-		(stroke
-			(width 0)
-			(type default)
-		)
-	)
-	(wire
-		(pts
 			(xy 257.81 95.25) (xy 257.81 97.79)
 		)
@@
 	(wire
 		(pts
-			(xy 21.59 74.93) (xy 41.91 74.93)
-		)
-		(stroke
-			(width 0)
-			(type default)
-		)
-	)
-	(wire
-		(pts
 			(xy 256.54 62.23) (xy 265.43 62.23)
 		)
@@
 	(wire
 		(pts
+			(xy 16.51 64.77) (xy 41.91 64.77)
+		)
+		(stroke
+			(width 0)
+			(type default)
+		)
+	)
+	(wire
+		(pts
 			(xy 241.3 96.52) (xy 241.3 99.06)
 		)
@@
 	(wire
 		(pts
-			(xy 15.24 74.93) (xy 21.59 74.93)
+			(xy 15.24 74.93) (xy 41.91 74.93)
 		)
 		(stroke
@@
 	(wire
 		(pts
-			(xy 41.91 69.85) (xy 21.59 69.85)
+			(xy 41.91 69.85) (xy 15.24 69.85)
 		)
 		(stroke
@@
 	(wire
 		(pts
+			(xy 16.51 60.96) (xy 16.51 64.77)
+		)
+		(stroke
+			(width 0)
+			(type default)
+		)
+	)
+	(wire
+		(pts
 			(xy 262.89 80.01) (xy 262.89 81.28)
 		)
@@
 	(wire
 		(pts
-			(xy 21.59 69.85) (xy 21.59 74.93)
+			(xy 15.24 69.85) (xy 15.24 74.93)
 		)
 		(stroke
@@
 		)
 	)
+	(hierarchical_label "TF_CS"
+		(shape input)
+		(at 29.21 59.69 180)
+		(effects
+			(font
+				(size 1.27 1.27)
+			)
+			(justify right)
+		)
+	)
+	(hierarchical_label "SPI_MISO"
+		(shape input)
+		(at 29.21 72.39 180)
+		(effects
+			(font
+				(size 1.27 1.27)
+			)
+			(justify right)
+		)
+	)
+	(hierarchical_label "SPI_MOSI"
+		(shape input)
+		(at 29.21 62.23 180)
+		(effects
+			(font
+				(size 1.27 1.27)
+			)
+			(justify right)
+		)
+	)
 	(hierarchical_label "CAM_SDA"
 		(shape input)
 		(at 256.54 31.75 180)
+		(effects
+			(font
+				(size 1.27 1.27)
+			)
+			(justify right)
+		)
+	)
+	(hierarchical_label "SPICLK"
+		(shape input)
+		(at 29.21 67.31 180)
 		(effects
 			(font
@@
 	(symbol
 		(lib_id "power:VAA")
-		(at 22.86 64.77 0)
+		(at 16.51 60.96 0)
 		(unit 1)
 		(exclude_from_sim no)
@@
 		(dnp no)
 		(property "Reference" "#PWR022"
-			(at 22.86 68.58 0)
+			(at 16.51 64.77 0)
 			(effects
 				(font
@@
 		)
 		(property "Value" "VDD_3V3"
-			(at 22.86 61.468 0)
+			(at 16.51 57.658 0)
 			(effects
 				(font
@@
 		)
 		(property "Footprint" ""
-			(at 22.86 64.77 0)
+			(at 16.51 60.96 0)
 			(effects
 				(font
@@
 		)
 		(property "Datasheet" ""
-			(at 22.86 64.77 0)
+			(at 16.51 60.96 0)
 			(effects
 				(font
@@
 		)
 		(property "Description" "Power symbol creates a global label with name \"VAA\""
-			(at 22.86 64.77 0)
-			(effects
-				(font
+			(at 16.51 60.96 0)
+			(effects
+				(font
