File: CLOCK_IT/Display.kicad_sch (KiCad schematic)
At the start: 0 parts

Commit message: :construction:added LCD connector,, completed connections
Parts:
- added J1: Conn_2Rows-29Pins, Connector_PinHeader_2.54mm:PinHeader_1x14_P2.54mm_Vertical, symbol Connector_Generic:Conn_2Rows-29Pins
- added J2: Conn_2Rows-09Pins, Connector_PinHeader_2.54mm:PinHeader_1x04_P2.54mm_Vertical, symbol Connector_Generic:Conn_2Rows-09Pins
Connections:
- net LCD_CS: now also J1.23 (Pin_23)
- net LCD_Data: now also J1.19 (Pin_19)
- net LCD_LED: now also J1.13 (Pin_13)
- net LCD_RST: now also J1.21 (Pin_21)
- net SPICLK: now also J1.15 (Pin_15), J2.7 (Pin_7)
- net SPI_MISO: now also J1.11 (Pin_11), J2.5 (Pin_5)
- net SPI_MOSI: now also J1.17 (Pin_17), J2.3 (Pin_3)
- new net CS: J1.24 (Pin_24)
- new net DC: J1.20 (Pin_20)
- new net GND: J1.26 (Pin_26)
- new net LED: J1.14 (Pin_14)
- new net RESET: J1.22 (Pin_22)
- new net SCK: J1.16 (Pin_16)
- new net SDI<MOSI>: J1.18 (Pin_18)
- new net SDO<MISO>: J1.12 (Pin_12)
- new net SD_CLK: J2.8 (Pin_8)
- new net SD_CS: J2.1 (Pin_1), J2.2 (Pin_2)
- new net SD_MISO: J2.6 (Pin_6)
- new net SD_MOSI: J2.4 (Pin_4)
- new net T_CLK: J1.10 (Pin_10)
- new net T_CS: J1.8 (Pin_8)
- new net T_DEN: J1.6 (Pin_6)
- new net T_DO: J1.4 (Pin_4)
- new net T_IRQ: J1.2 (Pin_2)
- new net Touch_CLK: J1.9 (Pin_9)
- new net Touch_CS: J1.7 (Pin_7)
- new net Touch_DIN: J1.5 (Pin_5)
- new net Touch_DOUT: J1.3 (Pin_3)
- new net Touch_IRQ: J1.1 (Pin_1)
- new net VCC: J1.28 (Pin_28)
