File: CLOCK_IT/CLOCK_IT.kicad_sch (KiCad schematic)
At the start: 0 parts

Commit message: :chart_with_upwards_trend:added display page:chart_with_upwards_trend:
Other:
- added sheet Display (Display.kicad_sch)
Changed lines of the file:
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@@
+	)
+	(sheet
+		(at 39.37 80.01)
+		(size 34.29 29.21)
+		(exclude_from_sim no)
+		(in_bom yes)
+		(on_board yes)
+		(dnp no)
+		(fields_autoplaced yes)
+		(stroke
+			(width 0.1524)
+			(type solid)
+		)
+		(fill
+			(color 0 0 0 0.0000)
+		)
+		(property "Sheetname" "Display"
+			(at 39.37 79.2984 0)
+			(effects
+				(font
+					(size 1.27 1.27)
+				)
+				(justify left bottom)
+			)
+		)
+		(property "Sheetfile" "Display.kicad_sch"
+			(at 39.37 109.8046 0)
+			(effects
+				(font
+					(size 1.27 1.27)
+				)
+				(justify left top)
+			)
+		)
+		(instances
+			(project "CLOCK_IT"
+				(path "/6c8f4e2a-0be1-4eb1-92e1-07339040f4c9"
+					(page "5")
+				)
+			)
+		)
 	)
 	(sheet

Commit message: :construction:added Audio IC
Other:
- added sheet Audio (Audio.kicad_sch)
Changed lines of the file:
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@@
+	)
+	(sheet
+		(at 92.71 82.55)
+		(size 38.1 26.67)
+		(exclude_from_sim no)
+		(in_bom yes)
+		(on_board yes)
+		(dnp no)
+		(fields_autoplaced yes)
+		(stroke
+			(width 0.1524)
+			(type solid)
+		)
+		(fill
+			(color 0 0 0 0.0000)
+		)
+		(property "Sheetname" "Audio"
+			(at 92.71 81.8384 0)
+			(effects
+				(font
+					(size 1.27 1.27)
+				)
+				(justify left bottom)
+			)
+		)
+		(property "Sheetfile" "Audio.kicad_sch"
+			(at 92.71 109.8046 0)
+			(effects
+				(font
+					(size 1.27 1.27)
+				)
+				(justify left top)
+			)
+		)
+		(instances
+			(project "CLOCK_IT"
+				(path "/6c8f4e2a-0be1-4eb1-92e1-07339040f4c9"
+					(page "6")
+				)
+			)
+		)
 	)
 	(sheet
