File: CLOCK_IT/mcu.kicad_sch (KiCad schematic)
At the start: 30 parts, among them IC1 APS6404L-3SQR-SN, SW2 HX 3X4X2-2P-1.6N TACTILE SWIT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, U1 ESP32-S3R8, U2 W25Q128JVSIQ, U7 PCA9548APW,118

Commit message: :construction:added display tags
Connections:
- net Cam_D6: now also U1.43 (GPIO38); no longer U1.21 (XTAL_32K_P)
- net LCD_CS: now reaches U1.13 (GPIO8)
- net LCD_Data: now reaches U1.14 (GPIO9)
- net LCD_RST: now reaches U1.15 (GPIO10)
- new net LCD_LED: U1.21 (XTAL_32K_P)
Changed lines of the file:
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@@
+	(wire
+		(pts
+			(xy 152.4 77.47) (xy 163.83 77.47)
+		)
+		(stroke
+			(width 0)
+			(type default)
+		)
+	)
 	(wire
 		(pts
@@
 	(wire
 		(pts
+			(xy 152.4 80.01) (xy 163.83 80.01)
+		)
+		(stroke
+			(width 0)
+			(type default)
+		)
+	)
+	(wire
+		(pts
 			(xy 176.53 52.07) (xy 176.53 49.53)
 		)
@@
 	(wire
 		(pts
+			(xy 152.4 82.55) (xy 163.83 82.55)
+		)
+		(stroke
+			(width 0)
+			(type default)
+		)
+	)
+	(wire
+		(pts
 			(xy 157.48 39.37) (xy 157.48 41.91)
 		)
@@
 		(pts
 			(xy 73.66 177.8) (xy 83.82 177.8)
+		)
+		(stroke
+			(width 0)
+			(type default)
+		)
+	)
+	(wire
+		(pts
+			(xy 152.4 120.65) (xy 162.56 120.65)
 		)
 		(stroke
@@
 	)
 	(label "Cam_D6"
-		(at 92.71 74.93 0)
-		(effects
-			(font
-				(size 1.27 1.27)
-			)
-			(justify left bottom)
+		(at 162.56 120.65 180)
+		(effects
+			(font
+				(size 1.27 1.27)
+			)
+			(justify right bottom)
 		)
 	)
@@
 		)
 	)
-	(label "USB_D-"
+	(label "USB_DN"
 		(at 162.56 100.33 180)
 		(effects
@@
 		)
 	)
+	(hierarchical_label "SPI_MOSI"
+		(shape input)
+		(at 162.56 118.11 0)
+		(effects
+			(font
+				(size 1.27 1.27)
+			)
+			(justify left)
+		)
+	)
 	(hierarchical_label "USB_DN"
 		(shape input)
@@
 		)
 	)
+	(hierarchical_label "SPI_MISO"
+		(shape input)
+		(at 162.56 113.03 0)
+		(effects
+			(font
+				(size 1.27 1.27)
+			)
+			(justify left)
+		)
+	)
 	(hierarchical_label "AXP_SCL"
 		(shape input)
@@
 		)
 	)
+	(hierarchical_label "LCD_CS"
+		(shape input)
+		(at 163.83 77.47 0)
+		(effects
+			(font
+				(size 1.27 1.27)
+			)
+			(justify left)
+		)
+	)
+	(hierarchical_label "LCD_RST"
+		(shape input)
+		(at 163.83 82.55 0)
+		(effects
+			(font
+				(size 1.27 1.27)
+			)
+			(justify left)
+		)
+	)
 	(hierarchical_label "USB_DP"
 		(shape input)
@@
 		)
 	)
+	(hierarchical_label "LCD_Data"
+		(shape input)
+		(at 163.83 80.01 0)
+		(effects
+			(font
+				(size 1.27 1.27)
+			)
+			(justify left)
+		)
+	)
 	(hierarchical_label "RTC_SCL"
 		(shape input)
@@
 		(effects
 			(font
+				(size 1.27 1.27)
+			)
+			(justify left)
+		)
+	)
+	(hierarchical_label "LCD_LED"
+		(shape input)
+		(at 92.71 74.93 180)
+		(effects
+			(font
+				(size 1.27 1.27)
+			)
+			(justify right)
+		)
+	)
+	(hierarchical_label "SPICLK"
+		(shape input)
+		(at 162.56 115.57 0)
+		(effects
+			(font

Commit message: :construction:added LCD connector,, completed connections
Connections:
- net Touch_CS: now reaches U1.10 (GPIO5)
- net Touch_IRQ: now reaches U1.9 (GPIO4)
Changed lines of the file:
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@@
+	(wire
+		(pts
+			(xy 152.4 67.31) (xy 165.1 67.31)
+		)
+		(stroke
+			(width 0)
+			(type default)
+		)
+	)
 	(wire
 		(pts
@@
 		(pts
 			(xy 233.68 57.15) (xy 233.68 52.07)
+		)
+		(stroke
+			(width 0)
+			(type default)
+		)
+	)
+	(wire
+		(pts
+			(xy 152.4 69.85) (xy 165.1 69.85)
 		)
 		(stroke
@@
 			)
 			(justify left bottom)
+		)
+	)
+	(hierarchical_label "SD_CS"
+		(shape input)
+		(at 176.53 63.5 0)
+		(effects
+			(font
+				(size 1.27 1.27)
+			)
+			(justify left)
 		)
 	)
@@
 		)
 	)
+	(hierarchical_label "TF_CS"
+		(shape input)
+		(at 176.53 60.96 0)
+		(effects
+			(font
+				(size 1.27 1.27)
+			)
+			(justify left)
+		)
+	)
 	(hierarchical_label "LCD_RST"
 		(shape input)
@@
 		)
 	)
+	(hierarchical_label "Touch_IRQ"
+		(shape input)
+		(at 165.1 67.31 0)
+		(effects
+			(font
+				(size 1.27 1.27)
+			)
+			(justify left)
+		)
+	)
 	(hierarchical_label "RTC_SCL"
 		(shape input)
@@
 		(effects
 			(font
+				(size 1.27 1.27)
+			)
+			(justify left)
+		)
+	)
+	(hierarchical_label "Touch_CS"
+		(shape input)
+		(at 165.1 69.85 0)
+		(effects
+			(font

Commit message: :construction: Dealing wih I2C and I2S
Connections:
- net SCLK_I2S: now reaches U1.23 (GPIO17)
- net Audio_SDA: now reaches U7.8 (SD2)
- net Audio_SCL: now reaches U7.9 (SC2)
Changed lines of the file:
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@@
+	(wire
+		(pts
+			(xy 208.28 129.54) (xy 213.36 129.54)
+		)
+		(stroke
+			(width 0)
+			(type default)
+		)
+	)
 	(wire
 		(pts
@@
 	(wire
 		(pts
+			(xy 152.4 95.25) (xy 163.83 95.25)
+		)
+		(stroke
+			(width 0)
+			(type default)
+		)
+	)
+	(wire
+		(pts
 			(xy 176.53 52.07) (xy 176.53 49.53)
 		)
@@
 		(pts
 			(xy 83.82 57.15) (xy 88.9 57.15)
+		)
+		(stroke
+			(width 0)
+			(type default)
+		)
+	)
+	(wire
+		(pts
+			(xy 208.28 132.08) (xy 213.36 132.08)
 		)
 		(stroke
@@
 		)
 	)
+	(hierarchical_label "Audio_SDA"
+		(shape input)
+		(at 208.28 129.54 180)
+		(effects
+			(font
+				(size 1.27 1.27)
+			)
+			(justify right)
+		)
+	)
 	(hierarchical_label "AXP_SDA"
 		(shape input)
@@
 		)
 	)
+	(hierarchical_label "Audio_CS"
+		(shape input)
+		(at 176.53 58.42 0)
+		(effects
+			(font
+				(size 1.27 1.27)
+			)
+			(justify left)
+		)
+	)
+	(hierarchical_label "SCL_I2S"
+		(shape input)
+		(at 163.83 90.17 0)
+		(effects
+			(font
+				(size 1.27 1.27)
+			)
+			(justify left)
+		)
+	)
 	(hierarchical_label "USB_DN"
 		(shape input)
@@
 		)
 	)
+	(hierarchical_label "SDA_I2S"
+		(shape input)
+		(at 163.83 92.71 0)
+		(effects
+			(font
+				(size 1.27 1.27)
+			)
+			(justify left)
+		)
+	)
 	(hierarchical_label "RTC_SCL"
 		(shape input)
@@
 		)
 	)
+	(hierarchical_label "SCLK_I2S"
+		(shape input)
+		(at 163.83 95.25 0)
+		(effects
+			(font
+				(size 1.27 1.27)
+			)
+			(justify left)
+		)
+	)
+	(hierarchical_label "Audio_SCL"
+		(shape input)
+		(at 208.28 132.08 180)
+		(effects
+			(font
+				(size 1.27 1.27)
+			)
+			(justify right)
+		)
+	)
