File: CLOCK_IT/Audio.kicad_sch (KiCad schematic)
At the start: 1 part, among them U8 ES8311

Commit message: :construction: Dealing wih I2C and I2S
Connections:
- net GND: now also U8.10 (AGND)
- net Audio_SCL: now reaches U8.1 (CCLK)
- net Audio_SDA: now reaches U8.19 (CDATA)
- net Audio_CS: now reaches U8.20 (CE)
- net SCLK_I2S: now reaches U8.6 (SCLK/DMIC_SCL)
- net SDA_I2S: now reaches U8.7 (ASDOUT)
- net SCL_I2S: now reaches U8.8 (LRCK)
Changed lines of the file:
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@@
 	(generator_version "9.0")
 	(paper "A4")
+	(wire
+		(pts
+			(xy 140.97 57.15) (xy 148.59 57.15)
+		)
+		(stroke
+			(width 0)
+			(type default)
+		)
+	)
+	(wire
+		(pts
+			(xy 80.01 69.85) (xy 85.09 69.85)
+		)
+		(stroke
+			(width 0)
+			(type default)
+		)
+	)
+	(wire
+		(pts
+			(xy 140.97 54.61) (xy 148.59 54.61)
+		)
+		(stroke
+			(width 0)
+			(type default)
+		)
+	)
+	(wire
+		(pts
+			(xy 80.01 67.31) (xy 85.09 67.31)
+		)
+		(stroke
+			(width 0)
+			(type default)
+		)
+	)
+	(wire
+		(pts
+			(xy 76.2 54.61) (xy 85.09 54.61)
+		)
+		(stroke
+			(width 0)
+			(type default)
+		)
+	)
+	(wire
+		(pts
+			(xy 80.01 72.39) (xy 85.09 72.39)
+		)
+		(stroke
+			(width 0)
+			(type default)
+		)
+	)
+	(wire
+		(pts
+			(xy 81.28 77.47) (xy 85.09 77.47)
+		)
+		(stroke
+			(width 0)
+			(type default)
+		)
+	)
+	(hierarchical_label "Audio_SCL"
+		(shape input)
+		(at 76.2 54.61 180)
+		(effects
+			(font
+				(size 1.27 1.27)
+			)
+			(justify right)
+		)
+	)
+	(hierarchical_label "Audio_SDA"
+		(shape input)
+		(at 148.59 57.15 0)
+		(effects
+			(font
+				(size 1.27 1.27)
+			)
+			(justify left)
+		)
+	)
+	(hierarchical_label "SCL_I2S"
+		(shape input)
+		(at 80.01 72.39 180)
+		(effects
+			(font
+				(size 1.27 1.27)
+			)
+			(justify right)
+		)
+	)
+	(hierarchical_label "SCLK_I2S"
+		(shape input)
+		(at 80.01 67.31 180)
+		(effects
+			(font
+				(size 1.27 1.27)
+			)
+			(justify right)
+		)
+	)
+	(hierarchical_label "Audio_CS"
+		(shape input)
+		(at 148.59 54.61 0)
+		(effects
+			(font
+				(size 1.27 1.27)
+			)
+			(justify left)
+		)
+	)
+	(hierarchical_label "SDA_I2S"
+		(shape input)
+		(at 80.01 69.85 180)
+		(effects
+			(font
+				(size 1.27 1.27)
+			)
+			(justify right)
+		)
+	)
 	(symbol
 		(lib_id "ES8311:ES8311")
@@
 	(symbol
 		(lib_id "power:GND")
-		(at 72.39 66.04 0)
+		(at 52.07 66.04 0)
 		(unit 1)
 		(exclude_from_sim no)
@@
 		(fields_autoplaced yes)
 		(property "Reference" "#PWR087"
-			(at 72.39 72.39 0)
+			(at 52.07 72.39 0)
 			(effects
 				(font
@@
 		)
 		(property "Value" "GND"
-			(at 72.39 71.12 0)
+			(at 52.07 71.12 0)
 			(effects
 				(font
@@
 		)
 		(property "Footprint" ""
-			(at 72.39 66.04 0)
+			(at 52.07 66.04 0)
 			(effects
 				(font
@@
 		)
 		(property "Datasheet" ""
-			(at 72.39 66.04 0)
+			(at 52.07 66.04 0)
 			(effects
 				(font
@@
 		)
 		(property "Description" "Power symbol creates a global label with name \"GND\" , ground"
-			(at 72.39 66.04 0)
+			(at 52.07 66.04 0)
 			(effects
 				(font
@@
 	(symbol
 		(lib_id "power:+3.3V")
-		(at 72.39 63.5 0)
+		(at 52.07 63.5 0)
 		(unit 1)
 		(exclude_from_sim no)
@@
 		(fields_autoplaced yes)
 		(property "Reference" "#PWR089"
-			(at 72.39 67.31 0)
+			(at 52.07 67.31 0)
 			(effects
 				(font
@@
 		)
 		(property "Value" "+3.3V"
-			(at 72.39 58.42 0)
+			(at 52.07 58.42 0)
 			(effects
 				(font
@@
 		)
 		(property "Footprint" ""
-			(at 72.39 63.5 0)
+			(at 52.07 63.5 0)
 			(effects
 				(font
@@
 		)
 		(property "Datasheet" ""
-			(at 72.39 63.5 0)
+			(at 52.07 63.5 0)
 			(effects
 				(font
@@
 		)
 		(property "Description" "Power symbol creates a global label with name \"+3.3V\""
-			(at 72.39 63.5 0)
+			(at 52.07 63.5 0)
 			(effects
 				(font
@@
 	(symbol
 		(lib_id "power:+3.3V")
-		(at 153.67 54.61 0)
+		(at 151.13 45.72 0)
 		(unit 1)
 		(exclude_from_sim no)
@@
 		(fields_autoplaced yes)
 		(property "Reference" "#PWR088"
-			(at 153.67 58.42 0)
+			(at 151.13 49.53 0)
 			(effects
 				(font
@@
 		)
 		(property "Value" "+3.3V"
-			(at 153.67 49.53 0)
+			(at 151.13 40.64 0)
 			(effects
 				(font
@@
 		)
 		(property "Footprint" ""
-			(at 153.67 54.61 0)
+			(at 151.13 45.72 0)
 			(effects
 				(font
@@
 		)
 		(property "Datasheet" ""
-			(at 153.67 54.61 0)
+			(at 151.13 45.72 0)
 			(effects
 				(font
@@
 		)
 		(property "Description" "Power symbol creates a global label with name \"+3.3V\""
-			(at 153.67 54.61 0)
+			(at 151.13 45.72 0)
 			(effects
 				(font
@@
 					(unit 1)
 				)
+			)
+		)
+	)
+	(symbol
+		(lib_id "power:GND")
+		(at 81.28 77.47 0)
+		(unit 1)
+		(exclude_from_sim no)
+		(in_bom yes)
+		(on_board yes)
+		(dnp no)
+		(fields_autoplaced yes)
+		(property "Reference" "#PWR090"
+			(at 81.28 83.82 0)
+			(effects
+				(font
+					(size 1.27 1.27)
+				)
+				(hide yes)
+			)
+		)
+		(property "Value" "GND"
+			(at 81.28 82.55 0)
+			(effects
+				(font
+					(size 1.27 1.27)
+				)
+			)
+		)
+		(property "Footprint" ""
+			(at 81.28 77.47 0)
+			(effects
+				(font
+					(size 1.27 1.27)
+				)
+				(hide yes)
+			)
+		)
+		(property "Datasheet" ""
+			(at 81.28 77.47 0)
+			(effects
+				(font
+					(size 1.27 1.27)
+				)
+				(hide yes)
+			)
+		)
+		(property "Description" "Power symbol creates a global label with name \"GND\" , ground"
+			(at 81.28 77.47 0)
+			(effects
+				(font
+					(size 1.27 1.27)
+				)
+				(hide yes)
+			)
+		)
+		(pin "1"
+		)
+		(instances
+			(project "CLOCK_IT"
+				(path "/6c8f4e2a-0be1-4eb1-92e1-07339040f4c9/854cfcf1-ae94-4a60-897d-29a1713dda3e"
+					(reference "#PWR090")
+					(unit 1)
+				)

Commit message: :construction: lable setting for speaker and mic
Parts:
- added C37, C38: 12pF, Capacitor_SMD:C_01005_0402Metric, symbol Device:C
- added C45: 0.1uF, symbol Device:C
- added R13: 2K2, symbol Device:R
- added R14: 100K, symbol Device:R
- added Y3: ABS07-32.768KHZ-T, Crystal:Crystal_SMD_5032-2Pin_5.0x3.2mm, symbol Device:Crystal
Connections:
- net +3.3V: now also U8.4 (DVDD)
- net GND: now also U8.5 (DGND), C37.2, C38.2
- net Speaker_OUTP: now reaches U8.12 (OUTP)
- net Speaker_OUTN: now reaches U8.13 (OUTN)
- net DACVREF: now reaches U8.14 (DACVREF)
- net ADCVREF: now reaches U8.15 (ADCVREF)
- net VMID: now reaches U8.16 (VMID)
- net MIC1N: now reaches U8.17 (MIC1N)
- net MIC1P: now reaches U8.18 (MIC1P/DMIC_SDA)
- net MCLK: now reaches U8.2 (MCLK)
- net MCLK: now also C38.1, Y3.1
- new net: C37.1, Y3.2
